File: CanSnif/CanSnif.kicad_pcb (KiCad board)
At the start: 4 copper layers, 50 x 50 mm, 65 parts, among them J1 JST_XH, J2 JST_XH, J3 Pin_Header, J4 USB_C_Receptacle_USB2.0_16P, J5 104031-0811, U1 STM32U575RGT6, U2 TJA1051T-3, U3 LDL212PV33R, U4 TPD6E05U06RVZ, U5 USBLC6-2SC6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

Commit message: Updated the Silkscreen
Parts:
- added G***: LOGO, LOGO, B.Cu at (38.4, 122.4)
- added kibuzzard-69AC87A2: G***, kibuzzard-69AC87A2, B.Cu at (38.4, 128.9)
- moved G*** 29.0 mm to (65.1, 137.8)
- moved G*** 2.00 mm to (38.6, 138.7)
- moved kibuzzard-69AC8543 0.68 mm to (36.7, 151.5)

Commit message: added battery orientation warning
Parts:
- added kibuzzard-69AC8A77: G***, kibuzzard-69AC8A77, B.Cu at (37.1, 150.9)
- moved kibuzzard-69AC8543 35.8 mm to (72.5, 151.8)
- moved G*** 0.70 mm to (60.3, 125.4)
- moved kibuzzard-69AC84C5 0.69 mm to (59.5, 133.7)
