File: CanSnif/Design Files/CanSnif.kicad_pcb (KiCad board)
At the start: 4 copper layers, 50 x 50 mm, 68 parts, among them J1 JST_XH, J2 JST_XH, J3 Pin_Header, J4 USB_C_Receptacle_USB2.0_16P, J5 104031-0811, U1 STM32U575RGT6, U2 TJA1051T-3, U3 LDL212PV33R, U4 TPD6E05U06RVZ, U5 USBLC6-2SC6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

Commit message: Finish
Parts:
- moved U4 0.08 mm to (55.5, 128.0)
Connections:
- R2 pad 1: SDMMC1_DAT0 -> SDMMC1_DAT2
- U1 pad 50: unconnected-(U1-PA15-Pad50) -> SDMMC1_SW
- U4 pad 1: Net-(J5-DAT2) -> SDMMC1_DAT2
- U4 pad 11: Net-(J5-CMD) -> SDMMC1_CMD
- U4 pad 12: Net-(J5-CLK) -> SDMMC1_CK
- U4 pad 14: Net-(J5-DAT2) -> SDMMC1_DAT2
- U4 pad 2: Net-(J5-CD/DAT3) -> SDMMC1_DAT3
- U4 pad 3: Net-(J5-CLK) -> SDMMC1_CK
- U4 pad 4: Net-(J5-CMD) -> SDMMC1_CMD
- U4 pad 6: Net-(J5-DAT1) -> SDMMC1_DAT1
- U4 pad 9: Net-(J5-DAT1) -> SDMMC1_DAT1
Routing:
- net SDMMC1_DAT0: track 38.8 -> 18.3 mm, vias 2 -> 0
- net SDMMC1_DAT2: track 2.78 -> 23.3 mm, vias 0 -> 2
- net SDMMC1_SW: track 11.2 -> 31.4 mm
- net GND: vias 327 -> 441
