File: CanSnif/Design Files/CanSnif.kicad_sch (KiCad schematic)
At the start: 59 parts, among them J1 JST_XH, J2 JST_XH, J3 Pin_Header, J4 USB_C_Receptacle_USB2.0_16P, J5 104031-0811, U1 STM32U575RGT6, U2 TJA1051T-3, U3 LDL212PV33R, U4 TPD6E05U06RVZ, U5 USBLC6-2SC6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

Commit message: Finish
Connections:
- net SDMMC1_SW: now also U1.50 (PA15)
Other:
- moved on the sheet: J2
Changed lines of the file:
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@@
 	(rectangle
 		(start 110.49 133.35)
-		(end 173.99 195.58)
+		(end 176.53 195.58)
 		(stroke
 			(width 0)
@@
 	(wire
 		(pts
+			(xy 34.29 96.52) (xy 41.91 96.52)
+		)
+		(stroke
+			(width 0)
+			(type default)
+		)
+	)
+	(wire
+		(pts
 			(xy 50.8 138.43) (xy 53.34 138.43)
 		)
@@
 	(wire
 		(pts
+			(xy 154.94 165.1) (xy 157.48 165.1)
+		)
+		(stroke
+			(width 0)
+			(type default)
+		)
+	)
+	(wire
+		(pts
 			(xy 38.1 81.28) (xy 38.1 86.36)
 		)
@@
 	(wire
 		(pts
-			(xy 106.68 99.06) (xy 104.14 99.06)
+			(xy 113.03 99.06) (xy 107.95 99.06)
 		)
 		(stroke
@@
 	(wire
 		(pts
-			(xy 30.48 43.18) (xy 41.91 43.18)
-		)
-		(stroke
-			(width 0)
-			(type default)
-		)
-	)
-	(wire
-		(pts
 			(xy 54.61 163.83) (xy 57.15 163.83)
 		)
@@
 	(wire
 		(pts
-			(xy 44.45 138.43) (xy 48.26 138.43)
+			(xy 34.29 139.7) (xy 48.26 139.7)
 		)
 		(stroke
@@
 	(wire
 		(pts
+			(xy 107.95 96.52) (xy 113.03 96.52)
+		)
+		(stroke
+			(width 0)
+			(type default)
+		)
+	)
+	(wire
+		(pts
 			(xy 119.38 185.42) (xy 119.38 187.96)
 		)
@@
 	(wire
 		(pts
+			(xy 153.67 73.66) (xy 161.29 73.66)
+		)
+		(stroke
+			(width 0)
+			(type default)
+		)
+	)
+	(wire
+		(pts
 			(xy 156.21 87.63) (xy 156.21 88.9)
 		)
@@
 	(wire
 		(pts
-			(xy 104.14 93.98) (xy 104.14 96.52)
+			(xy 107.95 93.98) (xy 107.95 96.52)
 		)
 		(stroke
@@
 	(wire
 		(pts
+			(xy 80.01 78.74) (xy 77.47 78.74)
+		)
+		(stroke
+			(width 0)
+			(type default)
+		)
+	)
+	(wire
+		(pts
 			(xy 81.28 175.26) (xy 76.2 175.26)
 		)
@@
 	(wire
 		(pts
-			(xy 34.29 96.52) (xy 41.91 96.52)
-		)
-		(stroke
-			(width 0)
-			(type default)
-		)
-	)
-	(wire
-		(pts
 			(xy 36.83 83.82) (xy 35.56 83.82)
 		)
@@
 	(wire
 		(pts
-			(xy 39.37 55.88) (xy 41.91 55.88)
+			(xy 154.94 162.56) (xy 157.48 162.56)
 		)
 		(stroke
@@
 	(wire
 		(pts
-			(xy 34.29 99.06) (xy 41.91 99.06)
+			(xy 39.37 55.88) (xy 41.91 55.88)
 		)
 		(stroke
@@
 	(wire
 		(pts
-			(xy 115.57 115.57) (xy 115.57 119.38)
+			(xy 34.29 99.06) (xy 41.91 99.06)
 		)
 		(stroke
@@
 	(wire
 		(pts
-			(xy 85.09 30.48) (xy 90.17 30.48)
+			(xy 115.57 115.57) (xy 115.57 119.38)
 		)
 		(stroke
@@
 	(wire
 		(pts
-			(xy 153.67 64.77) (xy 158.75 64.77)
+			(xy 85.09 30.48) (xy 90.17 30.48)
 		)
 		(stroke
@@
 	(wire
 		(pts
-			(xy 147.32 114.3) (xy 147.32 116.84)
+			(xy 153.67 64.77) (xy 158.75 64.77)
 		)
 		(stroke
@@
 	(wire
 		(pts
-			(xy 153.67 73.66) (xy 161.29 73.66)
+			(xy 147.32 114.3) (xy 147.32 116.84)
 		)
 		(stroke
@@
 	(wire
 		(pts
-			(xy 106.68 96.52) (xy 104.14 96.52)
-		)
-		(stroke
-			(width 0)
-			(type default)
-		)
-	)
-	(wire
-		(pts
 			(xy 83.82 156.21) (xy 83.82 160.02)
 		)
@@
 	(wire
 		(pts
-			(xy 165.1 154.94) (xy 162.56 154.94)
+			(xy 162.56 154.94) (xy 165.1 154.94)
 		)
 		(stroke
@@
 	(wire
 		(pts
+			(xy 30.48 43.18) (xy 41.91 43.18)
+		)
+		(stroke
+			(width 0)
+			(type default)
+		)
+	)
+	(wire
+		(pts
 			(xy 139.7 48.26) (xy 137.16 48.26)
 		)
@@
 	(wire
 		(pts
-			(xy 44.45 139.7) (xy 44.45 138.43)
+			(xy 34.29 142.24) (xy 34.29 139.7)
 		)
 		(stroke
@@
 	(wire
 		(pts
-			(xy 104.14 99.06) (xy 104.14 100.33)
+			(xy 107.95 99.06) (xy 107.95 100.33)
 		)
 		(stroke
@@
 	(wire
 		(pts
+			(xy 48.26 139.7) (xy 48.26 138.43)
+		)
+		(stroke
+			(width 0)
+			(type default)
+		)
+	)
+	(wire
+		(pts
 			(xy 53.34 158.75) (xy 53.34 161.29)
 		)
@@
 	(global_label "USB_OTG_FS_D-"
 		(shape input)
-		(at 154.94 162.56 0)
+		(at 157.48 162.56 0)
 		(fields_autoplaced yes)
 		(effects
@@
 		)
 		(property "Intersheetrefs" "${INTERSHEET_REFS}"
-			(at 173.3466 162.56 0)
+			(at 175.8866 162.56 0)
 			(effects
 				(font
@@
 	(global_label "SDMMC1_DAT0"
 		(shape input)
-		(at 44.45 139.7 180)
+		(at 34.29 142.24 180)
 		(fields_autoplaced yes)
 		(effects
@@
 		)
 		(property "Intersheetrefs" "${INTERSHEET_REFS}"
-			(at 28.0997 139.7 0)
+			(at 17.9397 142.24 0)
 			(effects
 				(font
@@
 		)
 	)
+	(global_label "SDMMC1_SW"
+		(shape input)
+		(at 80.01 78.74 0)
+		(fields_autoplaced yes)
+		(effects
+			(font
+				(size 1.27 1.27)
+			)
+			(justify left)
+		)
+		(property "Intersheetrefs" "${INTERSHEET_REFS}"
+			(at 94.4855 78.74 0)
+			(effects
+				(font
+					(size 1.27 1.27)
+				)
+				(justify left)
+				(hide yes)
+			)
+		)
+	)
 	(global_label "FDCAN_S"
 		(shape input)
@@
 	(global_label "USB_OTG_FS_D+"
 		(shape input)
-		(at 154.94 165.1 0)
+		(at 157.48 165.1 0)
 		(fields_autoplaced yes)
 		(effects
@@
 		)
 		(property "Intersheetrefs" "${INTERSHEET_REFS}"
-			(at 173.3466 165.1 0)
+			(at 175.8866 165.1 0)
 			(effects
 				(font
@@
 	(symbol
 		(lib_id "power:+5V")
-		(at 104.14 93.98 0)
+		(at 107.95 93.98 0)
 		(unit 1)
 		(exclude_from_sim no)
@@
 		(fields_autoplaced yes)
 		(property "Reference" "#PWR011"
-			(at 104.14 97.79 0)
+			(at 107.95 97.79 0)
 			(effects
 				(font
@@
 		)
 		(property "Value" "+5V"
-			(at 104.14 88.9 0)
+			(at 107.95 88.9 0)
 			(effects
 				(font
@@
 		)
 		(property "Footprint" ""
-			(at 104.14 93.98 0)
+			(at 107.95 93.98 0)
 			(effects
 				(font
@@
 		)
 		(property "Datasheet" ""
-			(at 104.14 93.98 0)
+			(at 107.95 93.98 0)
 			(effects
 				(font
@@
 		)
 		(property "Description" "Power symbol creates a global label with name \"+5V\""
-			(at 104.14 93.98 0)
+			(at 107.95 93.98 0)
 			(effects
 				(font
@@
 	(symbol
 		(lib_id "power:GND")
-		(at 104.14 100.33 0)
+		(at 107.95 100.33 0)
 		(unit 1)
 		(exclude_from_sim no)
@@
 		(dnp no)
 		(property "Reference" "#PWR012"
-			(at 104.14 106.68 0)
+			(at 107.95 106.68 0)
 			(effects
 				(font
@@
 		)
 		(property "Value" "GND"
-			(at 107.188 102.616 0)
+			(at 110.998 102.616 0)
 			(effects
 				(font
@@
 		)
 		(property "Footprint" ""
-			(at 104.14 100.33 0)
+			(at 107.95 100.33 0)
 			(effects
 				(font
@@
 		)
 		(property "Datasheet" ""
-			(at 104.14 100.33 0)
+			(at 107.95 100.33 0)
 			(effects
 				(font
@@
 		)
 		(property "Description" "Power symbol creates a global label with name \"GND\" , ground"
-			(at 104.14 100.33 0)
+			(at 107.95 100.33 0)
 			(effects
 				(font
@@
 	(symbol
 		(lib_id "Connector:Conn_01x02_Socket")
-		(at 111.76 96.52 0)
+		(at 118.11 96.52 0)
 		(unit 1)
 		(exclude_from_sim no)
@@
 		(dnp no)
 		(property "Reference" "J2"
-			(at 113.03 96.5199 0)
+			(at 119.38 96.5199 0)
 			(effects
 				(font
@@
 		)
 		(property "Value" "JST_XH"
-			(at 113.03 99.0599 0)
+			(at 119.38 99.0599 0)
 			(effects
 				(font
@@
 		)
 		(property "Footprint" "Connector_JST:JST_PH_S2B-PH-SM4-TB_1x02-1MP_P2.00mm_Horizontal"
-			(at 111.76 96.52 0)
+			(at 118.11 96.52 0)
 			(effects
 				(font
@@
 		)
 		(property "Datasheet" "~"
-			(at 111.76 96.52 0)
+			(at 118.11 96.52 0)
 			(effects
 				(font
@@
 		)
 		(property "Description" "Generic connector, single row, 01x02, script generated"
-			(at 111.76 96.52 0)
+			(at 118.11 96.52 0)
 			(effects
 				(font
@@
 		)
 		(property "Value" "USBLC6-2SC6"
-			(at 166.624 160.274 0)
+			(at 156.718 157.226 0)
 			(effects
 				(font
@@
 		(dnp no)
 		(property "Reference" "U2"
-			(at 116.332 51.816 0)
+			(at 127 61.976 0)
 			(effects
 				(font
@@
 		)
 		(property "Value" "TJA1051T-3"
-			(at 116.332 54.356 0)
+			(at 124.714 64.77 0)
 			(effects
 				(font
